File: hardware/power.sch (KiCad schematic (older format))
At the start: 38 parts, among them J4 USB_C_Receptacle, U10 TLV62568DBV, U4 XC6206P302MR, U7 TLV62568DBV, U8 TLV62568DBV, U9 TLV62568DBV

Commit message: Actually comitted the translation
Other:
- note added: "Alternative switcher: DIO6011"
Changed lines of the file:
@@
 	1    0    0    -1
 $EndComp
+Text Notes 9300 1700 0    50   ~ 0
+Alternative switcher: DIO6011
 $EndSCHEMATC

Commit message: Move Y1 to top-layer
Parts:
- R30: value 0 -> 0R
Changed lines of the file:
@@
 P 1900 2000
 F 0 "R30" V 2000 2000 50  0000 C CNN
-F 1 "0" V 1900 2000 50  0000 C CNN
+F 1 "0R" V 1900 2000 50  0000 C CNN
 F 2 "Resistor_SMD:R_0603_1608Metric" V 1830 2000 50  0001 C CNN
 F 3 "~" H 1900 2000 50  0001 C CNN
