File: hardware/moonpi_v2.kicad_pcb (KiCad board)
At the start: 4 copper layers, 60 x 60 mm, 121 parts, among them J1 JAE_SIM_Card_SF72S006, J11 Micro_SD_Card, J2 UART, J3 Bus_PCI_Express_Mini, J4 USB_C_Receptacle, J8 HR911105_RJ45, SW2 SW_MEC_5G, U1 AllwinnerV3S, U10 TLV62568DBV, U2 CH340C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

Commit message: Fixed filenames
Parts:
- J8: footprint balmer:HR911105_RJ45 -> moonpi:HR911105_RJ45
- U1: footprint balmer:eLQFP-128_14x14mm_P0.4mm -> moonpi:eLQFP-128_14x14mm_P0.4mm
Changed lines of the file:
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@@
     )
   )
-  (module balmer:eLQFP-128_14x14mm_P0.4mm (layer F.Cu)
+  (module moonpi:eLQFP-128_14x14mm_P0.4mm (layer F.Cu)
     (at 110.3 116.45 90)
     (descr "LQFP, 128 Pin (https://www.renesas.com/eu/en/package-image/pdf/outdrawing/q128.14x14.pdf), generated with kicad-footprint-generator ipc_gullwing_generator.py")
@@
     )
   )
-  (module balmer:HR911105_RJ45 (layer F.Cu)
+  (module moonpi:HR911105_RJ45 (layer F.Cu)
     (at 108.8 81.35 180)
     (tags HR911105_RJ45)
