File: hardware/moonpi_v2.sch (KiCad schematic (older format))
At the start: 38 parts, among them U1 AllwinnerV3S

Commit message: Fixed filenames
Parts:
- U1: footprint balmer:eLQFP-128_14x14mm_P0.4mm -> moonpi:eLQFP-128_14x14mm_P0.4mm; symbol balmer_allwinner_v3s_v2-rescue:AllwinnerV3S-balmer -> moonpi_v2-rescue:AllwinnerV3S-moonpi
Changed lines of the file:
@@
 $EndComp
 $Comp
-L balmer_allwinner_v3s_v2-rescue:AllwinnerV3S-balmer U1
+L moonpi_v2-rescue:AllwinnerV3S-moonpi U1
 U 1 1 5F2097DC
 P 4450 4700
 F 0 "U1" H 4450 4950 50  0000 L CNN
 F 1 "AllwinnerV3S" H 4300 4800 50  0000 L CNN
-F 2 "balmer:eLQFP-128_14x14mm_P0.4mm" H 4550 4750 50  0001 C CNN
+F 2 "moonpi:eLQFP-128_14x14mm_P0.4mm" H 4550 4750 50  0001 C CNN
 F 3 "" H 3400 5150 50  0001 C CNN
 	1    4450 4700
