File: hardware/moonpi.sch (KiCad schematic (older format))
At the start: 38 parts, among them U1 AllwinnerV3S

Commit message: Fixed filename verioning
Parts:
- U1: symbol moonpi_v2-rescue:AllwinnerV3S-moonpi -> moonpi-rescue:AllwinnerV3S-moonpi
Changed lines of the file:
@@
 $EndComp
 $Comp
-L moonpi_v2-rescue:AllwinnerV3S-moonpi U1
+L moonpi-rescue:AllwinnerV3S-moonpi U1
 U 1 1 5F2097DC
 P 4450 4700

Commit message: Changed USB series termination resistors values to zero-ohm
Parts:
- R24, R25: value 33R -> 0R
Changed lines of the file:
@@
 P 4600 1050
 F 0 "R24" V 4600 950 50  0000 L CNN
-F 1 "33R" V 4500 1000 50  0000 L CNN
+F 1 "0R" V 4500 1000 50  0000 L CNN
 F 2 "Resistor_SMD:R_0603_1608Metric" V 4530 1050 50  0001 C CNN
 F 3 "~" H 4600 1050 50  0001 C CNN
@@
 P 4700 1050
 F 0 "R25" V 4700 950 50  0000 L CNN
-F 1 "33R" V 4800 1000 50  0000 L CNN
+F 1 "0R" V 4800 1000 50  0000 L CNN
 F 2 "Resistor_SMD:R_0603_1608Metric" V 4630 1050 50  0001 C CNN
 F 3 "~" H 4700 1050 50  0001 C CNN
